File: src/Schematics for board/Schematics for board.sch (KiCad schematic (older format))
At the start: 18 parts

Commit message: Added some photos for schematics
Parts:
- removed JP?: Water Detector, symbol Jumper:SolderJumper_2_Open
- removed R?: 10k, symbol Device:R_US
- removed RV?: R_POT, symbol Device:R_POT
Connections:
- net A0: no longer names the net of A?.19 (A0)
- net A6: no longer names the net of A?.25 (A6)
- no-connect marks 12 -> 20
Other:
- note added: "Blue LED"
- note added: "x1 Digital\nGND"
- note removed: "Pot(entiometer)"
- note removed: "RGB LED"
- note removed: "Rariable Resistor\nx1 Analog"
- note removed: "x3 PWM\nGND"
- moved on the sheet: BZ?, D?, M?, R?, RV?, SW?, U?
